File: OdomBoard.sch (EAGLE design)
At the start: 36 parts, among them CN1 8P8C-LED, J1 EP2.5-4-SIDE, J2 EP2.5-4-SIDE, J3 EP2.5-4-SIDE, SW1 SWITCH_TACTILETOP, U1 STM32F103C8, U2 NCV7351D1E, U6 MC34063AD, U7 XC6206

Commit message: First Version
Parts:
- removed C14, C17: 22u, rcl:CPOL-EUE2-5
- removed C15: 220p, rcl:C-EUC0603
- removed D8: (no value), diode:DIODE-SOD123
- removed JP1: (no value), pinhead:PINHD-2X4
- removed L1: 220u, l_ysk:L5852
- removed R21: 3.6k, rcl:R-EU_R0603
- removed R22: 1.2k, rcl:R-EU_R0603
- removed R23: 0.68, rcl:R-EU_R1206
- removed U6: MC34063AD, mc34063:MC34063AD
- added C11: 10u, rcl:C-EUC1210
- added C8: EEEHA1E220P, rcl:CPOL-EU153CLV-0605
- added C9: 100n, rcl:C-EUC0603
- added H1, H2, H3, H4: MOUNT-HOLE3.0, CRS_EAGLE_Lib:MOUNT-HOLE3.0
- added IC3: MPU-9250_MOD, CRS_EAGLE_Lib:MPU-9250_MOD
- added R3, R5: 4.7k, rcl:R-EU_R0603
- added SV1: (no value), con-lstb:MA04-1
- added U13: 78L05F, linear:78L05F
Connections:
- net CANH renamed CAN_PAIR_P
- net CANL renamed CAN_PAIR_N
- removed net +24V: C14.+, CN1.A-G, F1.1, R23.1, U6.VCC
- removed net N$13: R23.2, U6.DC, U6.IS, U6.SWC
- removed net N$14: D8.C, L1.1, U6.SWE
- removed net N$15: C15.1, U6.TC
- removed net N$17: R21.1, R22.2, U6.FB
- removed net UART_RX: JP1.1
- removed net UART_TX: JP1.3
- new net +12V: C8.+, CN1.A-G, F1.1, U13.VI
- new net MPU_INT: IC3.INT, U1.PA12
- new net N$3: IC3.AUX_DA, R3.1
- new net N$4: IC3.AUX_CL, R5.1
- net +3V3: now also IC3.VDD, IC3.VDDIO, R3.2, R5.2, SV1.4; no longer JP1.8
- net +5V: now also C11.2, C9.1, U13.VO; no longer C17.+, JP1.5, L1.2, R21.2
- net GNDIO: now also C11.1, C8.-, C9.2, IC3.GND, SV1.1, U13.GND, U13.GND@1; no longer C14.-, C15.2, C17.-, D8.A, JP1.2, JP1.7, R22.1, U6.GND
- net SPI1_CS: now also IC3.CS
- net SPI1_MISO: now also IC3.SDO
- net SPI1_MOSI: now also IC3.SDI
- net SPI1_SCK: now also IC3.SCLK
- net SWCLK: now also SV1.2; no longer JP1.4
- net SWDIO: now also SV1.3; no longer JP1.6
- net TIM3_CH1: now also J3.3, U1.PA6; no longer J3.4, U1.PA7
- net TIM3_CH2: now also J3.4, U1.PA7; no longer J3.3, U1.PA6
